File: USB_Hub.kicad_pcb (KiCad board)
At the start: 2 copper layers, 65 x 30 mm, 36 parts, among them J1 USB, J2 USB_OTG, SW1 SW_RST, U1 GL850G, Y1 12Mhz

Commit message: rev2
Connections:
- R3 pad 2: /USB5V -> /USBGND
Routing:
- net /USB5V: track 74.6 -> 71.6 mm
- net /USBGND: track 116.5 -> 119.1 mm
Other:
- board text added: "C1,C4,C5,C13 100n C3 1u C8,C12 33p R6 5.1k R7 10k R2 100"
- board text removed: "C20,C23,C25,C35 100n C22 1u C26,C27 22p R15 5.1k R16 10k R19 100"
Changed lines of the file:
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@@
     (thickness 1.6)
     (drawings 22)
-    (tracks 407)
+    (tracks 415)
     (zones 0)
     (modules 36)
@@
       (net 21 "Net-(R3-Pad1)"))
     (pad 2 smd rect (at 0.95 0) (size 0.7 1.3) (layers F.Cu F.Paste F.Mask)
-      (net 6 /USB5V))
+      (net 3 /USBGND))
     (model ${KISYS3DMOD}/Resistors_SMD.3dshapes/R_0805.wrl
       (at (xyz 0 0 0))
@@
   (gr_line (start 82 84) (end 23 84) (angle 90) (layer Edge.Cuts) (width 0.15))
   (gr_line (start 85 111) (end 85 87) (angle 90) (layer Edge.Cuts) (width 0.15))
-  (gr_text "C20,C23,C25,C35 100n\nC22 1u\nC26,C27 22p\nR15 5.1k\nR16 10k\nR19 100\n" (at 49.784 97.536) (layer B.SilkS)
+  (gr_text "C1,C4,C5,C13 100n\nC3 1u\nC8,C12 33p\nR6 5.1k\nR7 10k\nR2 100\n" (at 49.784 97.536) (layer B.SilkS)
     (effects (font (size 1 1) (thickness 0.15)) (justify mirror))
   )
@@
   (segment (start 30.8 85.1) (end 33.62 85.1) (width 0.25) (layer F.Cu) (net 2))
   (segment (start 33.62 85.1) (end 35.22 86.7) (width 0.25) (layer F.Cu) (net 2))
+  (segment (start 50.05 85) (end 50.71 85) (width 0.4) (layer F.Cu) (net 3) (status 400000))
+  (segment (start 50.9 85.19) (end 50.9 86.9) (width 0.4) (layer F.Cu) (net 3))
+  (segment (start 50.71 85) (end 50.9 85.19) (width 0.4) (layer F.Cu) (net 3))
   (segment (start 62.75 85.4) (end 66.55 85.4) (width 0.4) (layer F.Cu) (net 3))
   (segment (start 66.15 85.8) (end 66.55 85.4) (width 0.4) (layer F.Cu) (net 3))
@@
   (segment (start 66.4 101.4) (end 67.5 101.4) (width 0.4) (layer F.Cu) (net 5))
   (segment (start 30.5 104) (end 30 104) (width 0.25) (layer F.Cu) (net 5))
+  (segment (start 48.26 92.1) (end 49.505 92.1) (width 0.4) (layer B.Cu) (net 6))
+  (segment (start 53.1 88.505) (end 53.1 88.1) (width 0.4) (layer F.Cu) (net 6))
+  (segment (start 52.705 88.9) (end 53.1 88.505) (width 0.4) (layer F.Cu) (net 6))
+  (via (at 52.705 88.9) (size 0.6) (drill 0.4) (layers F.Cu B.Cu) (net 6))
+  (segment (start 49.505 92.1) (end 52.705 88.9) (width 0.4) (layer B.Cu) (net 6))
+  (segment (start 49.1 92.1) (end 48.26 92.1) (width 0.4) (layer B.Cu) (net 6))
+  (segment (start 48.26 92.1) (end 47.3 92.1) (width 0.4) (layer B.Cu) (net 6))
+  (via (at 47.3 92.1) (size 0.6) (drill 0.4) (layers F.Cu B.Cu) (net 6))
+  (segment (start 47.3 92.1) (end 47.2 92.2) (width 0.4) (layer F.Cu) (net 6))
+  (segment (start 47.2 92.2) (end 42.7 92.2) (width 0.4) (layer F.Cu) (net 6))
+  (via (at 42.7 92.2) (size 0.6) (drill 0.4) (layers F.Cu B.Cu) (net 6))
+  (segment (start 42.7 92.2) (end 41.1 93.8) (width 0.4) (layer B.Cu) (net 6))
+  (segment (start 41.1 93.8) (end 38.6 93.8) (width 0.4) (layer B.Cu) (net 6))
+  (segment (start 38.6 93.8) (end 37 95.4) (width 0.4) (layer B.Cu) (net 6))
+  (via (at 37 95.4) (size 0.6) (drill 0.4) (layers F.Cu B.Cu) (net 6))
   (segment (start 66 88.1) (end 65.9 88.1) (width 0.4) (layer F.Cu) (net 6))
+  (segment (start 66 88.1) (end 67.5 88.1) (width 0.4) (layer F.Cu) (net 6))
+  (segment (start 67.5 88.1) (end 68.4 87.2) (width 0.4) (layer F.Cu) (net 6))
+  (segment (start 68.4 87.2) (end 70.4 87.2) (width 0.4) (layer F.Cu) (net 6))
+  (segment (start 70.4 87.2) (end 72.6 89.4) (width 0.4) (layer F.Cu) (net 6))
+  (segment (start 72.6 89.4) (end 72.6 91) (width 0.4) (layer F.Cu) (net 6))
+  (segment (start 53.1 88.1) (end 56.1 88.1) (width 0.4) (layer F.Cu) (net 6))
+  (segment (start 65.9 88.1) (end 65.2 88.8) (width 0.4) (layer F.Cu) (net 6))
+  (segment (start 65.2 88.8) (end 56.8 88.8) (width 0.4) (layer F.Cu) (net 6))
   (segment (start 56.8 88.8) (end 56.1 88.1) (width 0.4) (layer F.Cu) (net 6))
-  (segment (start 65.2 88.8) (end 56.8 88.8) (width 0.4) (layer F.Cu) (net 6))
-  (segment (start 65.9 88.1) (end 65.2 88.8) (width 0.4) (layer F.Cu) (net 6))
   (segment (start 24.9 92.5) (end 28.5 92.5) (width 0.4) (layer F.Cu) (net 6))
   (segment (start 28.5 92.5) (end 30.8 94.8) (width 0.4) (layer F.Cu) (net 6))
-  (segment (start 50.05 85) (end 49.4 85) (width 0.4) (layer F.Cu) (net 6))
-  (via (at 37 95.4) (size 0.6) (drill 0.4) (layers F.Cu B.Cu) (net 6))
-  (segment (start 38.6 93.8) (end 37 95.4) (width 0.4) (layer B.Cu) (net 6))
-  (segment (start 41.1 93.8) (end 38.6 93.8) (width 0.4) (layer B.Cu) (net 6))
-  (segment (start 42.7 92.2) (end 41.1 93.8) (width 0.4) (layer B.Cu) (net 6))
-  (via (at 42.7 92.2) (size 0.6) (drill 0.4) (layers F.Cu B.Cu) (net 6))
-  (segment (start 47.2 92.2) (end 42.7 92.2) (width 0.4) (layer F.Cu) (net 6))
-  (segment (start 47.3 92.1) (end 47.2 92.2) (width 0.4) (layer F.Cu) (net 6))
-  (via (at 47.3 92.1) (size 0.6) (drill 0.4) (layers F.Cu B.Cu) (net 6))
-  (segment (start 49.1 92.1) (end 47.3 92.1) (width 0.4) (layer B.Cu) (net 6))
-  (via (at 49.1 92.1) (size 0.6) (drill 0.4) (layers F.Cu B.Cu) (net 6))
-  (segment (start 49.1 85.3) (end 49.1 92.1) (width 0.4) (layer F.Cu) (net 6))
-  (segment (start 49.4 85) (end 49.1 85.3) (width 0.4) (layer F.Cu) (net 6))
   (segment (start 38.975 97.9) (end 38.975 96.775) (width 0.4) (layer F.Cu) (net 6))
   (segment (start 38.975 96.775) (end 37.6 95.4) (width 0.4) (layer F.Cu) (net 6))
@@
   (segment (start 31.4 95.4) (end 30.8 94.8) (width 0.4) (layer F.Cu) (net 6))
   (segment (start 51.85 85) (end 52.4 85) (width 0.4) (layer F.Cu) (net 6))
+  (segment (start 52.8 87.8) (end 53.1 88.1) (width 0.4) (layer F.Cu) (net 6))
+  (segment (start 52.8 85.4) (end 52.8 87.8) (width 0.4) (layer F.Cu) (net 6))
   (segment (start 52.4 85) (end 52.8 85.4) (width 0.4) (layer F.Cu) (net 6))
-  (segment (start 52.8 85.4) (end 52.8 87.8) (width 0.4) (layer F.Cu) (net 6))
-  (segment (start 52.8 87.8) (end 53.1 88.1) (width 0.4) (layer F.Cu) (net 6))
-  (segment (start 53.1 88.1) (end 56.1 88.1) (width 0.4) (layer F.Cu) (net 6))
-  (segment (start 72.6 89.4) (end 72.6 91) (width 0.4) (layer F.Cu) (net 6))
-  (segment (start 70.4 87.2) (end 72.6 89.4) (width 0.4) (layer F.Cu) (net 6))
-  (segment (start 68.4 87.2) (end 70.4 87.2) (width 0.4) (layer F.Cu) (net 6))
-  (segment (start 67.5 88.1) (end 68.4 87.2) (width 0.4) (layer F.Cu) (net 6))
-  (segment (start 66 88.1) (end 67.5 88.1) (width 0.4) (layer F.Cu) (net 6))
-  (segment (start 50.05 85) (end 51.85 85) (width 0.4) (layer F.Cu) (net 6))
   (segment (start 72.6 91) (end 72.6 92) (width 0.25) (layer F.Cu) (net 6))
   (segment (start 72.6 92) (end 74.8 94.2) (width 0.25) (layer F.Cu) (net 6))
@@
   (segment (start 60.85 86.05) (end 62.1 87.3) (width 0.25) (layer F.Cu) (net 20))
   (segment (start 62.1 87.3) (end 64.1 87.3) (width 0.25) (layer F.Cu) (net 20))
-  (segment (start 40.275 90.7) (end 40.275 89.325) (width 0.25) (layer F.Cu) (net 21))
-  (segment (start 46.95 86.2) (end 48.15 85) (width 0.25) (layer F.Cu) (net 21))
-  (segment (start 43.4 86.2) (end 46.95 86.2) (width 0.25) (layer F.Cu) (net 21))
-  (segment (start 40.275 89.325) (end 43.4 86.2) (width 0.25) (layer F.Cu) (net 21))
+  (segment (start 46.355 86.36) (end 47.625 85.09) (width 0.25) (layer F.Cu) (net 21))
+  (segment (start 47.625 85.09) (end 48.06 85.09) (width 0.25) (layer F.Cu) (net 21) (status 800000))
+  (segment (start 48.06 85.09) (end 48.15 85) (width 0.25) (layer F.Cu) (net 21) (status C00000))
+  (segment (start 40.275 90.7) (end 40.275 89.265) (width 0.25) (layer F.Cu) (net 21) (status 400000))
+  (segment (start 45.085 86.36) (end 46.355 86.36) (width 0.25) (layer F.Cu) (net 21))
+  (segment (start 43.18 88.265) (end 45.085 86.36) (width 0.25) (layer F.Cu) (net 21))
+  (segment (start 41.275 88.265) (end 43.18 88.265) (width 0.25) (layer F.Cu) (net 21))
+  (segment (start 40.275 89.265) (end 41.275 88.265) (width 0.25) (layer F.Cu) (net 21))
   (segment (start 35.725 97.9) (end 35.725 99.775) (width 0.25) (layer F.Cu) (net 22))
   (segment (start 35.725 99.775) (end 36.05 100.1) (width 0.25) (layer F.Cu) (net 22))
