File: USB_Hub.sch (KiCad schematic (older format))
At the start: 34 parts, among them J1 USB, J2 USB_OTG, SW1 SW_RST, U1 GL850G, Y1 12Mhz

Commit message: rev2
Connections:
- net USB5V: no longer R3.2
- net USBGND: now also R3.2
Other:
- moved on the sheet: C1, C10, C11, C12, C13, C14, C15, C16, C2, C3, C4, C5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
